Commit message: minor fixes

File: config/fire_fighter.urdf (robot description, URDF)
Before this commit: robot fire_fighter, 2 links, 1 joints
Joints:
- joint ld06_joint: origin xyz=0 0 0.1 rpy=0 3.14 0 -> xyz=0 0 0.1 rpy=0 0 0

Commit message: laser is still rotated in Z axis, just no longer inverted

File: config/fire_fighter.urdf (robot description, URDF)
Before this commit: robot fire_fighter, 2 links, 1 joints
Joints:
- joint ld06_joint: origin xyz=0 0 0.1 rpy=0 0 0 -> xyz=0 0 0.1 rpy=0 0 3.14

Commit message: update urdf

File: config/fire_fighter.urdf (robot description, URDF)
Before this commit: robot fire_fighter, 2 links, 1 joints
Links:
- added link left_wheel_link; visual cylinder length=0.02032 radius=0.0365
- added link right_wheel_link; visual cylinder length=0.02032 radius=0.0365
- added link top_deck_link; visual mesh filename=package://fire_fighter/config/top_deck.stl scale=0.001 0.001 0.001
- link base_link: geometry visual box size=0.150 0.130 0.047
- link ld06_frame: geometry visual cylinder length=0.03 radius=0.017
Joints:
- added joint left_wheel_joint: type continuous, parent base_link, child left_wheel_link, origin xyz=0.0 0.077 0.0365 rpy=0 0 0, axis 0 1 0
- added joint right_wheel_joint: type continuous, parent base_link, child right_wheel_link, origin xyz=0.0 -0.077 0.0365 rpy=0 0 0, axis 0 1 0
- added joint top_deck_joint: type fixed, parent base_link, child top_deck_link, origin xyz=0 0 0.109 rpy=0 0 0
- joint ld06_joint: origin xyz=0 0 0.1 rpy=0 0 3.14 -> xyz=0 0 0.157 rpy=0 0 3.14
